File: acoustic-carrier-hw/acoustic-carrier-board/fpga-config-flash.kicad_sch (KiCad schematic)
At the start: 20 parts, among them IC1 ECP5-BGA256, J701 Conn_02x07_Odd_Even, J702 Conn_02x09_Odd_Even, U701 W25Q128JVS, U702 W25Q128JVS

Commit message: [carrier] Change connectors to PMOD, follow specifications, check gappropriate power conenctor
Parts:
- added J703, J704: Conn_02x06_Odd_Even, Connector_PinHeader_2.54mm:PinHeader_2x06_P2.54mm_Horizontal, symbol Connector_Generic:Conn_02x06_Odd_Even
Connections:
- net GND: now also J703.11 (Pin_11)
- net QSPI.CSPPIn1: now also J703.1 (Pin_1)
- net VCORE_3V3: now also J703.12 (Pin_12)
