File: acoustic-carrier-board/connectors.kicad_sch (KiCad schematic)
At the start: 2 parts, among them J704 PMOD_GPIO, J903 Conn_02x06_Odd_Even

Commit message: added step-files
Parts:
- J704: LCSC Part Number (none) -> C2897426; LPN C2897426 -> (none); MPN PM254-2-06-W-8.5 -> (none); Manufacturing Part Number (none) -> PM254-2-06-W-8.5
- J903: now left out of the parts list
Changed lines of the file:
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@@
 			)
 		)
-		(property "LPN" "C2897426"
+		(property "LCSC Part Number" "C2897426"
 			(at 115.57 64.77 0)
 			(effects
@@
 			)
 		)
-		(property "MPN" "PM254-2-06-W-8.5 "
-			(at 115.824 68.072 0)
+		(property "Manufacturing Part Number" "PM254-2-06-W-8.5 "
+			(at 115.57 64.77 0)
 			(effects
 				(font
@@
 		(unit 1)
 		(exclude_from_sim no)
-		(in_bom yes)
+		(in_bom no)
 		(on_board yes)
 		(dnp no)
