File: acoustic-carrier-board/fpga-dqbank-23.kicad_sch (KiCad schematic)
At the start: 11 parts, among them IC1 ECP5-BGA256

Commit message: added step-files
Parts:
- C501, C502, C508, C509, C510, C513: LCSC Part Number (none) -> C22435929; LPN C22435929 -> (none); MPN CGA0201X7R104K160ET -> (none); Manufacturing Part Number (none) -> CGA0201X7R104K160ET
- C503, C512: LCSC Part Number (none) -> C23733; LPN C23733 -> (none); MPN CL05A475MP5NRNC -> (none); Manufacturing Part Number (none) -> CL05A475MP5NRNC
- C507, C511: LCSC Part Number (none) -> C285010; LPN C285010 -> (none); MPN 0201B103K250NT -> (none); Manufacturing Part Number (none) -> 0201B103K250NT
- IC1: LCSC Part Number (none) -> C1521614; LPN C1521614 -> (none); MPN LFE5U-25F-6BG256C -> (none); Manufacturing Part Number (none) -> LFE5U-25F-6BG256C
Changed lines of the file:
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@@
-			)
-		)
-		(property "LPN" "C22435929"
-			(at 114.3 33.02 0)
-			(effects
-				(font
-					(size 1.27 1.27)
-				)
-				(hide yes)
-			)
-		)
-		(property "MPN" "CGA0201X7R104K160ET "
-			(at 114.3 33.02 0)
-			(effects
-				(font
-					(size 1.27 1.27)
-				)
-				(hide yes)
 			)
 		)
@@
 			)
 		)
-		(property "Check_prices" ""
+		(property "LCSC Part Number" "C22435929"
+			(at 114.3 33.02 0)
+			(effects
+				(font
+					(size 1.27 1.27)
+				)
+				(hide yes)
+			)
+		)
+		(property "Manufacturing Part Number" "CGA0201X7R104K160ET "
 			(at 114.3 33.02 0)
 			(effects
@@
 			)
 		)
-		(property "LPN" "C285010"
-			(at 240.03 33.02 0)
-			(effects
-				(font
-					(size 1.27 1.27)
-				)
-				(hide yes)
-			)
-		)
-		(property "MPN" "0201B103K250NT"
-			(at 240.03 33.02 0)
-			(effects
-				(font
-					(size 1.27 1.27)
-				)
-				(hide yes)
-			)
-		)
 		(property "Availability" ""
 			(at 240.03 33.02 0)
@@
 			)
 		)
-		(property "Check_prices" ""
+		(property "LCSC Part Number" "C285010"
+			(at 240.03 33.02 0)
+			(effects
+				(font
+					(size 1.27 1.27)
+				)
+				(hide yes)
+			)
+		)
+		(property "Manufacturing Part Number" "0201B103K250NT"
 			(at 240.03 33.02 0)
 			(effects
@@
 			)
 		)
-		(property "LPN" "C1521614"
-			(at 106.68 -33.02 0)
-			(effects
-				(font
-					(size 1.27 1.27)
-				)
-				(justify left)
-				(hide yes)
-			)
-		)
-		(property "MPN" "LFE5U-25F-6BG256C "
-			(at 178.816 97.536 0)
+		(property "LCSC Part Number" "C1521614"
+			(at 198.12 97.79 0)
+			(effects
+				(font
+					(size 1.27 1.27)
+				)
+				(hide yes)
+			)
+		)
+		(property "Manufacturing Part Number" "LFE5U-25F-6BG256C "
+			(at 198.12 97.79 0)
 			(effects
 				(font
@@
 			)
 		)
-		(property "LPN" "C285010"
-			(at 64.77 29.21 0)
-			(effects
-				(font
-					(size 1.27 1.27)
-				)
-				(hide yes)
-			)
-		)
-		(property "MPN" "0201B103K250NT"
-			(at 64.77 29.21 0)
-			(effects
-				(font
-					(size 1.27 1.27)
-				)
-				(hide yes)
-			)
-		)
 		(property "Availability" ""
 			(at 64.77 29.21 0)
@@
 			)
 		)
-		(property "Check_prices" ""
+		(property "LCSC Part Number" "C285010"
+			(at 64.77 29.21 0)
+			(effects
+				(font
+					(size 1.27 1.27)
+				)
+				(hide yes)
+			)
+		)
+		(property "Manufacturing Part Number" "0201B103K250NT"
 			(at 64.77 29.21 0)
 			(effects
@@
 			)
 		)
-		(property "LPN" "C22435929"
-			(at 231.14 33.02 0)
-			(effects
-				(font
-					(size 1.27 1.27)
-				)
-				(hide yes)
-			)
-		)
-		(property "MPN" "CGA0201X7R104K160ET "
-			(at 231.14 33.02 0)
-			(effects
-				(font
-					(size 1.27 1.27)
-				)
-				(hide yes)
-			)
-		)
 		(property "Availability" ""
 			(at 231.14 33.02 0)
@@
 			)
 		)
-		(property "Check_prices" ""
+		(property "LCSC Part Number" "C22435929"
+			(at 231.14 33.02 0)
+			(effects
+				(font
+					(size 1.27 1.27)
+				)
+				(hide yes)
+			)
+		)
+		(property "Manufacturing Part Number" "CGA0201X7R104K160ET "
 			(at 231.14 33.02 0)
 			(effects
@@
 			)
 		)
-		(property "LPN" "C22435929"
-			(at 222.25 33.02 0)
-			(effects
-				(font
-					(size 1.27 1.27)
-				)
-				(hide yes)
-			)
-		)
-		(property "MPN" "CGA0201X7R104K160ET "
-			(at 222.25 33.02 0)
-			(effects
-				(font
-					(size 1.27 1.27)
-				)
-				(hide yes)
-			)
-		)
 		(property "Availability" ""
 			(at 222.25 33.02 0)
@@
 			)
 		)
-		(property "Check_prices" ""
+		(property "LCSC Part Number" "C22435929"
+			(at 222.25 33.02 0)
+			(effects
+				(font
+					(size 1.27 1.27)
+				)
+				(hide yes)
+			)
+		)
+		(property "Manufacturing Part Number" "CGA0201X7R104K160ET "
 			(at 222.25 33.02 0)
 			(effects
@@
 			)
 		)
-		(property "LPN" "C23733"
-			(at 124.46 33.02 0)
-			(effects
-				(font
-					(size 1.27 1.27)
-				)
-				(hide yes)
-			)
-		)
-		(property "MPN" "CL05A475MP5NRNC"
-			(at 124.46 33.02 0)
-			(effects
-				(font
-					(size 1.27 1.27)
-				)
-				(hide yes)
-			)
-		)
 		(property "Availability" ""
 			(at 124.46 33.02 0)
@@
 			)
 		)
-		(property "Check_prices" ""
+		(property "LCSC Part Number" "C23733"
+			(at 124.46 33.02 0)
+			(effects
+				(font
+					(size 1.27 1.27)
+				)
+				(hide yes)
+			)
+		)
+		(property "Manufacturing Part Number" "CL05A475MP5NRNC"
 			(at 124.46 33.02 0)
 			(effects
@@
 			)
 		)
-		(property "LPN" "C1521614"
-			(at -34.29 -29.21 0)
-			(effects
-				(font
-					(size 1.27 1.27)
-				)
-				(justify left)
-				(hide yes)
-			)
-		)
-		(property "MPN" "LFE5U-25F-6BG256C "
-			(at 37.846 101.346 0)
+		(property "LCSC Part Number" "C1521614"
+			(at 57.15 101.6 0)
+			(effects
+				(font
+					(size 1.27 1.27)
+				)
+				(hide yes)
+			)
+		)
+		(property "Manufacturing Part Number" "LFE5U-25F-6BG256C "
+			(at 57.15 101.6 0)
 			(effects
 				(font
@@
 			)
 		)
-		(property "LPN" "C22435929"
-			(at 72.39 29.21 0)
-			(effects
-				(font
-					(size 1.27 1.27)
-				)
-				(hide yes)
-			)
-		)
-		(property "MPN" "CGA0201X7R104K160ET "
-			(at 72.39 29.21 0)
-			(effects
-				(font
-					(size 1.27 1.27)
-				)
-				(hide yes)
-			)
-		)
 		(property "Availability" ""
 			(at 72.39 29.21 0)
@@
 			)
 		)
-		(property "Check_prices" ""
+		(property "LCSC Part Number" "C22435929"
+			(at 72.39 29.21 0)
+			(effects
+				(font
+					(size 1.27 1.27)
+				)
+				(hide yes)
+			)
+		)
+		(property "Manufacturing Part Number" "CGA0201X7R104K160ET "
 			(at 72.39 29.21 0)
 			(effects
@@
 			)
 		)
-		(property "LPN" "C22435929"
-			(at 102.87 33.02 0)
-			(effects
-				(font
-					(size 1.27 1.27)
-				)
-				(hide yes)
-			)
-		)
-		(property "MPN" "CGA0201X7R104K160ET "
-			(at 102.87 33.02 0)
-			(effects
-				(font
-					(size 1.27 1.27)
-				)
-				(hide yes)
-			)
-		)
 		(property "Availability" ""
 			(at 102.87 33.02 0)
@@
 			)
 		)
-		(property "Check_prices" ""
+		(property "LCSC Part Number" "C22435929"
+			(at 102.87 33.02 0)
+			(effects
+				(font
+					(size 1.27 1.27)
+				)
+				(hide yes)
+			)
+		)
+		(property "Manufacturing Part Number" "CGA0201X7R104K160ET "
 			(at 102.87 33.02 0)
 			(effects
@@
 			)
 		)
-		(property "LPN" "C22435929"
-			(at 251.46 118.11 0)
-			(effects
-				(font
-					(size 1.27 1.27)
-				)
-				(hide yes)
-			)
-		)
-		(property "MPN" "CGA0201X7R104K160ET "
-			(at 251.46 118.11 0)
-			(effects
-				(font
-					(size 1.27 1.27)
-				)
-				(hide yes)
-			)
-		)
 		(property "Availability" ""
 			(at 251.46 118.11 0)
@@
 			)
 		)
-		(property "Check_prices" ""
+		(property "LCSC Part Number" "C22435929"
+			(at 251.46 118.11 0)
+			(effects
+				(font
+					(size 1.27 1.27)
+				)
+				(hide yes)
+			)
+		)
+		(property "Manufacturing Part Number" "CGA0201X7R104K160ET "
 			(at 251.46 118.11 0)
 			(effects
@@
 			)
 		)
-		(property "LPN" "C23733"
-			(at 247.65 33.02 0)
-			(effects
-				(font
-					(size 1.27 1.27)
-				)
-				(hide yes)
-			)
-		)
-		(property "MPN" "CL05A475MP5NRNC"
-			(at 247.65 33.02 0)
-			(effects
-				(font
-					(size 1.27 1.27)
-				)
-				(hide yes)
-			)
-		)
 		(property "Availability" ""
 			(at 247.65 33.02 0)
@@
 			)
 		)
-		(property "Check_prices" ""
+		(property "LCSC Part Number" "C23733"
 			(at 247.65 33.02 0)
 			(effects
+				(font
+					(size 1.27 1.27)
+				)
+				(hide yes)
+			)
+		)
+		(property "Manufacturing Part Number" "CL05A475MP5NRNC"
+			(at 247.65 33.02 0)
+			(effects
