File: acoustic-carrier-board/fpga-dqbank-67.kicad_sch (KiCad schematic)
At the start: 20 parts, among them IC1 ECP5-BGA256, SW602 SW_Push, SW603 SW_Push

Commit message: added step-files
Parts:
- C601, C604, C606, C612, C613: LCSC Part Number (none) -> C22435929; LPN C22435929 -> (none); MPN CGA0201X7R104K160ET -> (none); Manufacturing Part Number (none) -> CGA0201X7R104K160ET
- C602: LCSC Part Number (none) -> C285010; LPN C285010 -> (none); MPN 0201B103K250NT -> (none); Manufacturing Part Number (none) -> 0201B103K250NT
- C603, C611: LCSC Part Number (none) -> C23733; LPN C23733 -> (none); MPN CL05A475MP5NRNC -> (none); Manufacturing Part Number (none) -> CL05A475MP5NRNC
- D601, D602: LCSC Part Number (none) -> C2286; LPN C2286 -> (none); MPN KT-0603R -> (none); Manufacturing Part Number (none) -> KT-0603R
- IC1: LCSC Part Number (none) -> C1521614; LPN C1521614 -> (none); MPN LFE5U-25F-6BG256C -> (none); Manufacturing Part Number (none) -> LFE5U-25F-6BG256C
- R601, R603, R605, R607: LCSC Part Number (none) -> C25117; LPN C25117 -> (none); MPN 0402WGF4700TCE -> (none); Manufacturing Part Number (none) -> 0402WGF4700TCE
- R602: LCSC Part Number (none) -> C21189; LPN C21189 -> (none); MPN 0603WAF0000T5E -> (none); Manufacturing Part Number (none) -> 0603WAF0000T5E
- R604, R606: LCSC Part Number (none) -> C25900; LPN C25900 -> (none); MPN 0402WGF4701TCE -> (none); Manufacturing Part Number (none) -> 0402WGF4701TCE
- SW602, SW603: LCSC Part Number (none) -> C720477; LPN C720477 -> (none); MPN TS-1088-AR02016 -> (none); Manufacturing Part Number (none) -> TS-1088-AR02016
Changed lines of the file:
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@@
 			)
 		)
-		(property "LPN" "C23733"
-			(at 90.17 30.48 0)
-			(effects
-				(font
-					(size 1.27 1.27)
-				)
-				(hide yes)
-			)
-		)
-		(property "MPN" "CL05A475MP5NRNC"
+		(property "Availability" ""
 			(at 90.17 30.48 0)
 			(effects
@@
 			)
 		)
-		(property "Availability" ""
+		(property "LCSC Part Number" "C23733"
 			(at 90.17 30.48 0)
 			(effects
@@
 			)
 		)
-		(property "Check_prices" ""
+		(property "Manufacturing Part Number" "CL05A475MP5NRNC"
 			(at 90.17 30.48 0)
 			(effects
@@
 			)
 		)
-		(property "LPN" "C25900"
+		(property "LCSC Part Number" "C25900"
 			(at 73.66 172.72 0)
 			(effects
@@
 			)
 		)
-		(property "MPN" "0402WGF4701TCE"
+		(property "Manufacturing Part Number" "0402WGF4701TCE"
 			(at 73.66 172.72 0)
 			(effects
@@
 			)
 		)
-		(property "MPN" "0402WGF4700TCE"
+		(property "LCSC Part Number" "C25117"
 			(at 90.17 179.07 0)
 			(effects
@@
 			)
 		)
-		(property "LPN" "C25117"
+		(property "Manufacturing Part Number" "0402WGF4700TCE"
 			(at 90.17 179.07 0)
 			(effects
@@
 			)
 		)
-		(property "LPN" "C720477"
+		(property "LCSC Part Number" "C720477"
 			(at 81.28 179.07 90)
 			(effects
@@
 			)
 		)
-		(property "MPN" "TS-1088-AR02016"
+		(property "Manufacturing Part Number" "TS-1088-AR02016"
 			(at 81.28 179.07 90)
 			(effects
@@
 			)
 		)
-		(property "LPN" "C720477"
+		(property "LCSC Part Number" "C720477"
 			(at 41.91 179.07 90)
 			(effects
@@
 			)
 		)
-		(property "MPN" "TS-1088-AR02016"
+		(property "Manufacturing Part Number" "TS-1088-AR02016"
 			(at 41.91 179.07 90)
 			(effects
@@
 			)
 		)
-		(property "LPN" "C23733"
-			(at 264.16 36.83 0)
-			(effects
-				(font
-					(size 1.27 1.27)
-				)
-				(hide yes)
-			)
-		)
-		(property "MPN" "CL05A475MP5NRNC"
+		(property "Availability" ""
 			(at 264.16 36.83 0)
 			(effects
@@
 			)
 		)
-		(property "Availability" ""
+		(property "LCSC Part Number" "C23733"
 			(at 264.16 36.83 0)
 			(effects
@@
 			)
 		)
-		(property "Check_prices" ""
+		(property "Manufacturing Part Number" "CL05A475MP5NRNC"
 			(at 264.16 36.83 0)
 			(effects
@@
 			)
 		)
-		(property "LPN" "C1521614"
-			(at -46.99 -44.45 0)
+		(property "LCSC Part Number" "C1521614"
+			(at 44.45 86.36 0)
 			(effects
 				(font
 					(size 1.27 1.27)
 				)
-				(justify left)
 				(hide yes)
 			)
 		)
-		(property "MPN" "LFE5U-25F-6BG256C "
-			(at 25.146 86.106 0)
+		(property "Manufacturing Part Number" "LFE5U-25F-6BG256C "
+			(at 44.45 86.36 0)
 			(effects
 				(font
@@
 			)
 		)
-		(property "LPN" "C25900"
-			(at 31.75 171.45 0)
-			(effects
-				(font
-					(size 1.27 1.27)
-				)
-				(hide yes)
-			)
-		)
-		(property "MPN" "0402WGF4701TCE"
+		(property "Availability" ""
 			(at 31.75 171.45 0)
 			(effects
@@
 			)
 		)
-		(property "Availability" ""
+		(property "LCSC Part Number" "C25900"
 			(at 31.75 171.45 0)
 			(effects
@@
 			)
 		)
-		(property "Check_prices" ""
+		(property "Manufacturing Part Number" "0402WGF4701TCE"
 			(at 31.75 171.45 0)
 			(effects
@@
 			)
 		)
-		(property "LPN" "C21189"
-			(at 222.25 68.58 90)
-			(effects
-				(font
-					(size 1.27 1.27)
-				)
-				(hide yes)
-			)
-		)
-		(property "MPN" "0603WAF0000T5E"
+		(property "Availability" ""
 			(at 222.25 68.58 90)
 			(effects
@@
 			)
 		)
-		(property "Availability" ""
+		(property "LCSC Part Number" "C21189"
 			(at 222.25 68.58 90)
 			(effects
@@
 			)
 		)
-		(property "Check_prices" ""
+		(property "Manufacturing Part Number" "0603WAF0000T5E"
 			(at 222.25 68.58 90)
 			(effects
@@
 			)
 		)
-		(property "LPN" "C1521614"
-			(at 109.22 -45.72 0)
+		(property "LCSC Part Number" "C1521614"
+			(at 200.66 85.09 0)
 			(effects
 				(font
 					(size 1.27 1.27)
 				)
-				(justify left)
 				(hide yes)
 			)
 		)
-		(property "MPN" "LFE5U-25F-6BG256C "
-			(at 181.356 84.836 0)
+		(property "Manufacturing Part Number" "LFE5U-25F-6BG256C "
+			(at 200.66 85.09 0)
 			(effects
 				(font
@@
 			)
 		)
-		(property "LPN" "C22435929"
-			(at 102.87 30.48 0)
-			(effects
-				(font
-					(size 1.27 1.27)
-				)
-				(hide yes)
-			)
-		)
-		(property "MPN" "CGA0201X7R104K160ET "
+		(property "Availability" ""
 			(at 102.87 30.48 0)
 			(effects
@@
 			)
 		)
-		(property "Availability" ""
+		(property "LCSC Part Number" "C22435929"
 			(at 102.87 30.48 0)
 			(effects
@@
 			)
 		)
-		(property "Check_prices" ""
+		(property "Manufacturing Part Number" "CGA0201X7R104K160ET "
 			(at 102.87 30.48 0)
 			(effects
@@
 			)
 		)
-		(property "MPN" "0402WGF4700TCE"
+		(property "LCSC Part Number" "C25117"
 			(at 50.8 179.07 0)
 			(effects
@@
 			)
 		)
-		(property "LPN" "C25117"
+		(property "Manufacturing Part Number" "0402WGF4700TCE"
 			(at 50.8 179.07 0)
 			(effects
@@
 			)
 		)
-		(property "LPN" "C2286"
-			(at 115.57 167.64 90)
-			(effects
-				(font
-					(size 1.27 1.27)
-				)
-				(hide yes)
-			)
-		)
-		(property "MPN" "KT-0603R "
+		(property "Availability" ""
 			(at 115.57 167.64 90)
 			(effects
@@
 			)
 		)
-		(property "Availability" ""
-			(at 115.57 167.64 90)
+		(property "LCSC Part Number" "C2286"
+			(at 115.57 167.64 0)
 			(effects
 				(font
@@
 			)
 		)
-		(property "Check_prices" ""
-			(at 115.57 167.64 90)
+		(property "Manufacturing Part Number" "KT-0603R "
+			(at 115.57 167.64 0)
 			(effects
 				(font
@@
 			)
 		)
-		(property "LPN" "C22435929"
+		(property "LCSC Part Number" "C22435929"
 			(at 74.93 182.88 0)
 			(effects
@@
 			)
 		)
-		(property "MPN" "CGA0201X7R104K160ET "
+		(property "Manufacturing Part Number" "CGA0201X7R104K160ET "
 			(at 74.93 182.88 0)
 			(effects
@@
 			)
 		)
-		(property "LPN" "C2286"
-			(at 115.57 179.07 90)
-			(effects
-				(font
-					(size 1.27 1.27)
-				)
-				(hide yes)
-			)
-		)
-		(property "MPN" "KT-0603R "
+		(property "Availability" ""
 			(at 115.57 179.07 90)
 			(effects
@@
 			)
 		)
-		(property "Availability" ""
-			(at 115.57 179.07 90)
+		(property "LCSC Part Number" "C2286"
+			(at 115.57 179.07 0)
 			(effects
 				(font
@@
 			)
 		)
-		(property "Check_prices" ""
-			(at 115.57 179.07 90)
+		(property "Manufacturing Part Number" "KT-0603R "
+			(at 115.57 179.07 0)
 			(effects
 				(font
@@
 			)
 		)
-		(property "MPN" "0402WGF4700TCE"
+		(property "LCSC Part Number" "C25117"
 			(at 121.92 184.15 0)
 			(effects
@@
 			)
 		)
-		(property "LPN" "C25117"
+		(property "Manufacturing Part Number" "0402WGF4700TCE"
 			(at 121.92 184.15 0)
 			(effects
@@
 			)
 		)
-		(property "LPN" "C22435929"
-			(at 250.19 36.83 0)
-			(effects
-				(font
-					(size 1.27 1.27)
-				)
-				(hide yes)
-			)
-		)
-		(property "MPN" "CGA0201X7R104K160ET "
+		(property "Availability" ""
 			(at 250.19 36.83 0)
 			(effects
@@
 			)
 		)
-		(property "Availability" ""
+		(property "LCSC Part Number" "C22435929"
 			(at 250.19 36.83 0)
 			(effects
@@
 			)
 		)
-		(property "Check_prices" ""
+		(property "Manufacturing Part Number" "CGA0201X7R104K160ET "
 			(at 250.19 36.83 0)
 			(effects
@@
 			)
 		)
-		(property "LPN" "C22435929"
-			(at 96.52 30.48 0)
-			(effects
-				(font
-					(size 1.27 1.27)
-				)
-				(hide yes)
-			)
-		)
-		(property "MPN" "CGA0201X7R104K160ET "
+		(property "Availability" ""
 			(at 96.52 30.48 0)
 			(effects
@@
 			)
 		)
-		(property "Availability" ""
+		(property "LCSC Part Number" "C22435929"
 			(at 96.52 30.48 0)
 			(effects
@@
 			)
 		)
-		(property "Check_prices" ""
+		(property "Manufacturing Part Number" "CGA0201X7R104K160ET "
 			(at 96.52 30.48 0)
 			(effects
@@
 			)
 		)
-		(property "LPN" "C22435929"
+		(property "LCSC Part Number" "C22435929"
 			(at 33.02 182.88 0)
 			(effects
@@
 			)
 		)
-		(property "MPN" "CGA0201X7R104K160ET "
+		(property "Manufacturing Part Number" "CGA0201X7R104K160ET "
 			(at 33.02 182.88 0)
 			(effects
@@
 			)
 		)
-		(property "LPN" "C285010"
-			(at 256.54 36.83 0)
-			(effects
-				(font
-					(size 1.27 1.27)
-				)
-				(hide yes)
-			)
-		)
-		(property "MPN" "0201B103K250NT"
+		(property "Availability" ""
 			(at 256.54 36.83 0)
 			(effects
@@
 			)
 		)
-		(property "Availability" ""
+		(property "LCSC Part Number" "C285010"
 			(at 256.54 36.83 0)
 			(effects
@@
 			)
 		)
-		(property "Check_prices" ""
+		(property "Manufacturing Part Number" "0201B103K250NT"
 			(at 256.54 36.83 0)
 			(effects
@@
 			)
 		)
-		(property "MPN" "0402WGF4700TCE"
+		(property "LCSC Part Number" "C25117"
 			(at 121.92 171.45 0)
 			(effects
@@
 			)
 		)
-		(property "LPN" "C25117"
+		(property "Manufacturing Part Number" "0402WGF4700TCE"
 			(at 121.92 171.45 0)
 			(effects
