File: acoustic-carrier-board/fpga-power.kicad_sch (KiCad schematic)
At the start: 16 parts, among them IC1 ECP5-BGA256

Commit message: added step-files
Parts:
- C301, C302, C303, C304, C305, C306, C310, C311: LCSC Part Number (none) -> C22435929; LPN C22435929 -> (none); MPN CGA0201X7R104K160ET -> (none); Manufacturing Part Number (none) -> CGA0201X7R104K160ET
- C307, C308, C309: LCSC Part Number (none) -> C19702; LPN C19702 -> (none); MPN CL10A106KP8NNNC -> (none); Manufacturing Part Number (none) -> CL10A106KP8NNNC
- C312: LCSC Part Number (none) -> C23733; LPN C23733 -> (none); MPN CL05A475MP5NRNC -> (none); Manufacturing Part Number (none) -> CL05A475MP5NRNC
- C313: LCSC Part Number (none) -> C59461; LPN C59461 -> (none); MPN CL10A226MQ8NRNC -> (none); Manufacturing Part Number (none) -> CL10A226MQ8NRNC
- IC1: LCSC Part Number (none) -> C1521614; LPN C1521614 -> (none); MPN LFE5U-25F-6BG256C -> (none); Manufacturing Part Number (none) -> LFE5U-25F-6BG256C
- R301: LCSC Part Number (none) -> C17477; LPN C17477 -> (none); MPN 0805W8F0000T5E -> (none); Manufacturing Part Number (none) -> 0805W8F0000T5E
- TP207: now left out of the parts list
