File: acoustic-carrier-board/power.kicad_sch (KiCad schematic)
At the start: 73 parts, among them J201 Conn_02x06_Odd_Even, Q201 AO3401A, U201 TPS2121RUX, U202 TLV62569DBV, U203 TLV62569DBV, U204 TLV62569DBV, U205 TLV62569DBV, U206 OPA376xxDBV

Commit message: minor changes
Connections:
- net BP_5V: now also J201.1 (Pin_1), J201.11 (Pin_11), J201.3 (Pin_3), J201.5 (Pin_5), J201.7 (Pin_7), J201.9 (Pin_9); no longer J201.10 (Pin_10), J201.12 (Pin_12), J201.2 (Pin_2), J201.4 (Pin_4), J201.6 (Pin_6), J201.8 (Pin_8)
- net GND: now also J201.10 (Pin_10), J201.12 (Pin_12), J201.2 (Pin_2), J201.4 (Pin_4), J201.6 (Pin_6), J201.8 (Pin_8); no longer J201.1 (Pin_1), J201.11 (Pin_11), J201.3 (Pin_3), J201.5 (Pin_5), J201.7 (Pin_7), J201.9 (Pin_9)
Changed lines of the file:
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@@
 	)
 	(junction
-		(at 41.91 44.45)
-		(diameter 0)
-		(color 0 0 0 0)
-	)
-	(junction
 		(at 201.93 41.91)
 		(diameter 0)
@@
 	)
 	(junction
-		(at 29.21 41.91)
+		(at 45.72 266.7)
 		(diameter 0)
 		(color 0 0 0 0)
 	)
 	(junction
-		(at 45.72 266.7)
+		(at 29.21 41.91)
 		(diameter 0)
 		(color 0 0 0 0)
@@
 	)
 	(junction
-		(at 29.21 39.37)
+		(at 29.21 44.45)
 		(diameter 0)
 		(color 0 0 0 0)
@@
 	)
 	(junction
-		(at 29.21 46.99)
-		(diameter 0)
-		(color 0 0 0 0)
-	)
-	(junction
 		(at 87.63 241.3)
 		(diameter 0)
@@
 	)
 	(junction
+		(at 29.21 46.99)
+		(diameter 0)
+		(color 0 0 0 0)
+	)
+	(junction
+		(at 29.21 39.37)
+		(diameter 0)
+		(color 0 0 0 0)
+	)
+	(junction
+		(at 41.91 39.37)
+		(diameter 0)
+		(color 0 0 0 0)
+	)
+	(junction
+		(at 41.91 44.45)
+		(diameter 0)
+		(color 0 0 0 0)
+	)
+	(junction
 		(at 92.71 147.32)
 		(diameter 0)
@@
 	)
 	(junction
+		(at 41.91 41.91)
+		(diameter 0)
+		(color 0 0 0 0)
+	)
+	(junction
 		(at 25.4 243.84)
 		(diameter 0)
@@
 	)
 	(junction
-		(at 29.21 44.45)
-		(diameter 0)
-		(color 0 0 0 0)
-	)
-	(junction
-		(at 41.91 39.37)
-		(diameter 0)
-		(color 0 0 0 0)
-	)
-	(junction
-		(at 41.91 46.99)
-		(diameter 0)
-		(color 0 0 0 0)
-	)
-	(junction
 		(at 143.51 78.74)
 		(diameter 0)
@@
 	)
 	(junction
-		(at 41.91 41.91)
-		(diameter 0)
+		(at 66.04 134.62)
+		(diameter 1.016)
 		(color 0 0 0 0)
 	)
 	(junction
-		(at 66.04 134.62)
-		(diameter 1.016)
+		(at 41.91 46.99)
+		(diameter 0)
 		(color 0 0 0 0)
 	)
@@
 	(wire
 		(pts
+			(xy 29.21 36.83) (xy 29.21 39.37)
+		)
+		(stroke
+			(width 0)
+			(type default)
+		)
+	)
+	(wire
+		(pts
 			(xy 205.74 251.46) (xy 205.74 254)
 		)
@@
 	(wire
 		(pts
-			(xy 41.91 44.45) (xy 41.91 46.99)
-		)
-		(stroke
-			(width 0)
-			(type default)
-		)
-	)
-	(wire
-		(pts
 			(xy 52.07 137.16) (xy 49.53 137.16)
 		)
@@
 	(wire
 		(pts
-			(xy 41.91 39.37) (xy 41.91 40.64)
-		)
-		(stroke
-			(width 0)
-			(type default)
-		)
-	)
-	(wire
-		(pts
 			(xy 35.56 252.73) (xy 35.56 254)
 		)
@@
 	(wire
 		(pts
-			(xy 29.21 46.99) (xy 29.21 49.53)
+			(xy 29.21 40.64) (xy 29.21 41.91)
 		)
 		(stroke
@@
 	(wire
 		(pts
-			(xy 41.91 36.83) (xy 41.91 39.37)
-		)
-		(stroke
-			(width 0)
-			(type default)
-		)
-	)
-	(wire
-		(pts
 			(xy 194.31 146.05) (xy 194.31 143.51)
 		)
@@
 	(wire
 		(pts
+			(xy 41.91 39.37) (xy 41.91 40.64)
+		)
+		(stroke
+			(width 0)
+			(type default)
+		)
+	)
+	(wire
+		(pts
 			(xy 92.71 134.62) (xy 101.6 134.62)
 		)
@@
 	(wire
 		(pts
-			(xy 29.21 40.64) (xy 29.21 41.91)
-		)
-		(stroke
-			(width 0)
-			(type default)
-		)
-	)
-	(wire
-		(pts
 			(xy 73.66 41.91) (xy 73.66 46.99)
 		)
@@
 	(wire
 		(pts
-			(xy 29.21 36.83) (xy 29.21 39.37)
-		)
-		(stroke
-			(width 0)
-			(type default)
-		)
-	)
-	(wire
-		(pts
 			(xy 215.9 251.46) (xy 220.98 251.46)
 		)
@@
 	(wire
 		(pts
-			(xy 29.21 39.37) (xy 29.21 40.64)
-		)
-		(stroke
-			(width 0)
-			(type default)
-		)
-	)
-	(wire
-		(pts
 			(xy 55.88 193.04) (xy 53.34 193.04)
 		)
@@
 	(wire
 		(pts
-			(xy 41.91 46.99) (xy 41.91 49.53)
+			(xy 41.91 40.64) (xy 41.91 41.91)
 		)
 		(stroke
@@
 	(wire
 		(pts
+			(xy 41.91 44.45) (xy 41.91 46.99)
+		)
+		(stroke
+			(width 0)
+			(type default)
+		)
+	)
+	(wire
+		(pts
 			(xy 96.52 41.91) (xy 143.51 41.91)
 		)
@@
 	(wire
 		(pts
-			(xy 29.21 44.45) (xy 29.21 46.99)
-		)
-		(stroke
-			(width 0)
-			(type default)
-		)
-	)
-	(wire
-		(pts
 			(xy 95.25 254) (xy 100.33 254)
 		)
@@
 	(wire
 		(pts
+			(xy 41.91 46.99) (xy 41.91 49.53)
+		)
+		(stroke
+			(width 0)
+			(type default)
+		)
+	)
+	(wire
+		(pts
 			(xy 62.23 198.12) (xy 62.23 200.66)
 		)
@@
 	(wire
 		(pts
-			(xy 29.21 41.91) (xy 29.21 44.45)
-		)
-		(stroke
-			(width 0)
-			(type default)
-		)
-	)
-	(wire
-		(pts
 			(xy 92.71 143.51) (xy 92.71 147.32)
 		)
@@
 	(wire
 		(pts
-			(xy 41.91 41.91) (xy 41.91 44.45)
-		)
-		(stroke
-			(width 0)
-			(type default)
-		)
-	)
-	(wire
-		(pts
 			(xy 123.19 134.62) (xy 133.35 134.62)
 		)
@@
 	(wire
 		(pts
+			(xy 29.21 41.91) (xy 29.21 44.45)
+		)
+		(stroke
+			(width 0)
+			(type default)
+		)
+	)
+	(wire
+		(pts
 			(xy 60.96 134.62) (xy 66.04 134.62)
 		)
@@
 	(wire
 		(pts
+			(xy 29.21 44.45) (xy 29.21 46.99)
+		)
+		(stroke
+			(width 0)
+			(type default)
+		)
+	)
+	(wire
+		(pts
 			(xy 245.11 147.32) (xy 245.11 149.86)
 		)
@@
 	(wire
 		(pts
+			(xy 29.21 46.99) (xy 29.21 49.53)
+		)
+		(stroke
+			(width 0)
+			(type default)
+		)
+	)
+	(wire
+		(pts
 			(xy 101.6 134.62) (xy 104.14 134.62)
 		)
@@
 	(wire
 		(pts
+			(xy 41.91 41.91) (xy 41.91 44.45)
+		)
+		(stroke
+			(width 0)
+			(type default)
+		)
+	)
+	(wire
+		(pts
 			(xy 74.93 187.96) (xy 86.36 187.96)
 		)
@@
 	(wire
 		(pts
+			(xy 41.91 36.83) (xy 41.91 39.37)
+		)
+		(stroke
+			(width 0)
+			(type default)
+		)
+	)
+	(wire
+		(pts
 			(xy 41.91 40.64) (xy 73.66 40.64)
 		)
@@
 	(wire
 		(pts
-			(xy 41.91 40.64) (xy 41.91 41.91)
+			(xy 125.73 241.3) (xy 133.35 241.3)
 		)
 		(stroke
@@
 	(wire
 		(pts
-			(xy 125.73 241.3) (xy 133.35 241.3)
+			(xy 27.94 243.84) (xy 27.94 246.38)
 		)
 		(stroke
@@
 	(wire
 		(pts
-			(xy 27.94 243.84) (xy 27.94 246.38)
+			(xy 143.51 86.36) (xy 143.51 87.63)
 		)
 		(stroke
@@
 	(wire
 		(pts
-			(xy 143.51 86.36) (xy 143.51 87.63)
+			(xy 29.21 39.37) (xy 29.21 40.64)
 		)
 		(stroke
@@
 	(symbol
 		(lib_id "Connector_Generic:Conn_02x06_Odd_Even")
-		(at 34.29 41.91 0)
+		(at 36.83 41.91 0)
+		(mirror y)
 		(unit 1)
 		(exclude_from_sim no)
@@
 		(on_board yes)
 		(dnp no)
-		(fields_autoplaced yes)
 		(property "Reference" "J201"
 			(at 35.56 30.48 0)
@@
 		)
 		(property "Footprint" "Connector_PinSocket_2.54mm:PinSocket_2x06_P2.54mm_Vertical"
-			(at 34.29 41.91 0)
+			(at 36.83 41.91 0)
 			(effects
 				(font
@@
 		)
 		(property "Datasheet" "~"
-			(at 34.29 41.91 0)
+			(at 36.83 41.91 0)
 			(effects
 				(font
@@
 		)
 		(property "Description" "Generic connector, double row, 02x06, odd/even pin numbering scheme (row 1 odd numbers, row 2 even numbers), script generated (kicad-library-utils/schlib/autogen/connector/)"
-			(at 34.29 41.91 0)
+			(at 36.83 41.91 0)
 			(effects
 				(font
@@
 		)
 		(property "LPN" ""
-			(at 34.29 41.91 0)
+			(at 36.83 41.91 0)
 			(effects
 				(font
@@
 		)
 		(property "MPN" ""
-			(at 34.29 41.91 0)
+			(at 36.83 41.91 0)
 			(effects
 				(font

Commit message: added step-files
Parts:
- C201: LCSC Part Number (none) -> C2162244; LPN C2162244 -> (none); MPN APXE160ARA151MH80G -> (none); Manufacturing Part Number (none) -> APXE160ARA151MH80G
- C202, C225, C227, C228: LCSC Part Number (none) -> C22435929; LPN C22435929 -> (none); MPN CGA0201X7R104K160ET -> (none); Manufacturing Part Number (none) -> CGA0201X7R104K160ET
- C203, C209, C217, C219: LCSC Part Number (none) -> C32949; LPN C32949 -> (none); MPN CL05C100JB5NNNC -> (none); Manufacturing Part Number (none) -> CL05C100JB5NNNC
- C204, C205, C206, C210, C211, C214, C215, C220, C221, C222: LCSC Part Number (none) -> C19702; LPN C19702 -> (none); MPN CL10A106KP8NNNC -> (none); Manufacturing Part Number (none) -> CL10A106KP8NNNC
- C207, C212, C216, C223: LCSC Part Number (none) -> C28323; LPN C28323 -> (none); MPN CL21B105KBFNNNE -> (none); Manufacturing Part Number (none) -> CL21B105KBFNNNE
- C208, C213, C218, C224: LCSC Part Number (none) -> C23733; LPN C23733 -> (none); MPN CL05A475MP5NRNC -> (none); Manufacturing Part Number (none) -> CL05A475MP5NRNC
- C226: LCSC Part Number (none) -> C285010; LPN C285010 -> (none); MPN 0201B103K250NT -> (none); Manufacturing Part Number (none) -> 0201B103K250NT
- D201: LCSC Part Number (none) -> C19077443; LPN C19077443 -> (none); MPN BZT52C6V8S -> (none); Manufacturing Part Number (none) -> BZT52C6V8S
- J201, TP202, TP205, TP206, TP208, TP209, TP210: now left out of the parts list
- L201, L202, L203, L204: LCSC Part Number (none) -> C28642347; LPN C28642347 -> (none); MPN NR4018S2R2MT -> (none); Manufacturing Part Number (none) -> NR4018S2R2MT
- Q201: LCSC Part Number (none) -> C15127; LPN C15127 -> (none); MPN AO3401A -> (none); Manufacturing Part Number (none) -> AO3401A
- R201, R202: LCSC Part Number (none) -> C25900; LPN C25900 -> (none); MPN 0402WGF4701TCE -> (none); Manufacturing Part Number (none) -> 0402WGF4701TCE
- R203, R216, R225, R226: LCSC Part Number (none) -> C23352; LPN C23352 -> (none); MPN 0603WAF2402T5E -> (none); Manufacturing Part Number (none) -> 0603WAF2402T5E
- R204, R210, R211, R213: LCSC Part Number (none) -> C25803; LPN C25803 -> (none); MPN 0603WAF1003T5E -> (none); Manufacturing Part Number (none) -> 0603WAF1003T5E
- R205: LCSC Part Number (none) -> C22967; LPN C22967 -> (none); MPN 0603WAF2702T5E -> (none); Manufacturing Part Number (none) -> 0603WAF2702T5E
- R206, R212: LCSC Part Number (none) -> C31850; LPN C31850 -> (none); MPN 0603WAF2202T5E -> (none); Manufacturing Part Number (none) -> 0603WAF2202T5E
- R207, R227: LCSC Part Number (none) -> C23186; LPN C23186 -> (none); MPN 0603WAF5101T5E -> (none); Manufacturing Part Number (none) -> 0603WAF5101T5E
- R208, R209, R217: LCSC Part Number (none) -> C17477; LPN C17477 -> (none); MPN 0805W8F0000T5E -> (none); Manufacturing Part Number (none) -> 0805W8F0000T5E
- R215: LCSC Part Number (none) -> C23242; LPN C23242 -> (none); MPN 0603WAF7502T5E -> (none); Manufacturing Part Number (none) -> 0603WAF7502T5E
- R218: LCSC Part Number (none) -> C22984; LPN C22984 -> (none); MPN 0603WAF3002T5E -> (none); Manufacturing Part Number (none) -> 0603WAF3002T5E
- R219, R223: LCSC Part Number (none) -> C21190; LPN C21190 -> (none); MPN 0603WAF1001T5E -> (none); Manufacturing Part Number (none) -> 0603WAF1001T5E
- R220, R221: LCSC Part Number (none) -> C21189; LPN C21189 -> (none); MPN 0603WAF0000T5E -> (none); Manufacturing Part Number (none) -> 0603WAF0000T5E
- R222: LCSC Part Number (none) -> C22962; LPN C22962 -> (none); MPN 0603WAF2200T5E -> (none); Manufacturing Part Number (none) -> 0603WAF2200T5E
- R224: LCSC Part Number (none) -> 0603WAF1001T5E; LPN 0603WAF1001T5E -> (none); MPN C21190 -> (none); Manufacturing Part Number (none) -> C21190
- U201: LCSC Part Number (none) -> C2156025; LPN C2156025 -> (none); MPN TPS2121RUXT -> (none); Manufacturing Part Number (none) -> TPS2121RUXT
- U202, U203, U204, U205: LCSC Part Number (none) -> C141836; LPN C141836 -> (none); MPN TLV62569DBVR -> (none); Manufacturing Part Number (none) -> TLV62569DBVR
- U206: LCSC Part Number (none) -> C42134; LPN C42134 -> (none); MPN OPA376AIDBVR -> (none); Manufacturing Part Number (none) -> OPA376AIDBVR
