File: acoustic-carrier-board/analog-frontend.kicad_sch (KiCad schematic)
At the start: 101 parts, among them J1001 BWU.FL-IPEX1, J1002 BWU.FL-IPEX1, J1003 BWU.FL-IPEX1, J1004 BWU.FL-IPEX1, J1005 BWU.FL-IPEX1, J1006 BWU.FL-IPEX1, J1007 8P8C_Shielded, J1008 BWU.FL-IPEX1, J1009 BWU.FL-IPEX1, J1010 BWU.FL-IPEX1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

Commit message: added step-files
Parts:
- C1001, C1006, C1007, C1023: LCSC Part Number (none) -> C19702; LPN C19702 -> (none); MPN CL10A106KP8NNNC -> (none); Manufacturing Part Number (none) -> CL10A106KP8NNNC
- C1002, C1003, C1004, C1005, C1008, C1009, C1010, C1011, C1013, C1019, C1021, C1024, C1026, C1027: LCSC Part Number (none) -> C22435929; LPN C22435929 -> (none); MPN CGA0201X7R104K160ET -> (none); Manufacturing Part Number (none) -> CGA0201X7R104K160ET
- C1012, C1015, C1016: LCSC Part Number (none) -> C1634; LPN C1634 -> (none); MPN CL10C100JB8NNNC -> (none); Manufacturing Part Number (none) -> CL10C100JB8NNNC
- C1014: LCSC Part Number (none) -> C28323; LPN C28323 -> (none); MPN CL21B105KBFNNNE -> (none); Manufacturing Part Number (none) -> CL21B105KBFNNNE
- C1017, C1018, C1028, C1029: LCSC Part Number (none) -> C88136; LPN C88136 -> (none); MPN 0603B104J500NT -> (none); Manufacturing Part Number (none) -> 0603B104J500NT
- C1020: LCSC Part Number (none) -> C16772; LPN C16772 -> (none); MPN CL05B224KO5NNNC -> (none); Manufacturing Part Number (none) -> CL05B224KO5NNNC
- C1022, C1025: LCSC Part Number (none) -> C285010; LPN C285010 -> (none); MPN 0201B103K250NT -> (none); Manufacturing Part Number (none) -> 0201B103K250NT
- J1001, J1002, J1003, J1004, J1005, J1006, J1008, J1009, J1010, J1011: LCSC Part Number (none) -> C5137195; LPN C5137195 -> (none); MPN BWU.FL-IPEX1 -> (none); Manufacturing Part Number (none) -> BWU.FL-IPEX1
- J1007: LCSC Part Number (none) -> C708652; LPN C708652 -> (none); MPN RC01937 -> (none); Manufacturing Part Number (none) -> RC01937
- L1001: LCSC Part Number (none) -> C113030; LPN C113030 -> (none); MPN BLM18SG121TN1D -> (none); Manufacturing Part Number (none) -> BLM18SG121TN1D
- R1001, R1007, R1008, R1011, R1014, R1022, R1025, R1026, R1039, R1043: LCSC Part Number (none) -> C21189; LPN C21189 -> (none); MPN 0603WAF0000T5E -> (none); Manufacturing Part Number (none) -> 0603WAF0000T5E
- R1002, R1003, R1004, R1005: LCSC Part Number (none) -> C23179; LPN C23179 -> (none); MPN 0603WAF4700T5E -> (none); Manufacturing Part Number (none) -> 0603WAF4700T5E
- R1006, R1010, R1023, R1027, R1028, R1029: LCSC Part Number (none) -> C25804; LPN C25804 -> (none); MPN 0603WAF1002T5E -> (none); Manufacturing Part Number (none) -> 0603WAF1002T5E
- R1009, R1013, R1021, R1024, R1030, R1031, R1032: LCSC Part Number (none) -> C21190; LPN C21190 -> (none); MPN 0603WAF1001T5E -> (none); Manufacturing Part Number (none) -> 0603WAF1001T5E
- R1012, R1015, R1017, R1018, R1020: LCSC Part Number (none) -> C17168; LPN C17168 -> (none); MPN 0402WGF0000TCE -> (none); Manufacturing Part Number (none) -> 0402WGF0000TCE
- R1016, R1019: LCSC Part Number (none) -> C23182; LPN C23182 -> (none); MPN 0603WAF470JT5E -> (none); Manufacturing Part Number (none) -> 0603WAF470JT5E
- R1033: LCSC Part Number (none) -> C4275; LPN C4275 -> (none); MPN 0603WAF750JT5E -> (none); Manufacturing Part Number (none) -> 0603WAF750JT5E
- R1034, R1036, R1037: LCSC Part Number (none) -> 0603WAF1001T5E; LPN 0603WAF1001T5E -> (none); MPN C21190 -> (none); Manufacturing Part Number (none) -> C21190
- R1035: LCSC Part Number (none) -> C22843; LPN C22843 -> (none); MPN 0603WAF1501T5E -> (none); Manufacturing Part Number (none) -> 0603WAF1501T5E
- R1038: LCSC Part Number (none) -> C23162; LPN C23162 -> (none); MPN 0603WAF4701T5E -> (none); Manufacturing Part Number (none) -> 0603WAF4701T5E
- RJ1001: LCSC Part Number (none) -> C163507; LPN C163507 -> (none); MPN HR913550A -> (none); Manufacturing Part Number (none) -> HR913550A
- TP1001, TP1005, TP1011, TP1012: now left out of the parts list
- U1001: LCSC Part Number (none) -> C1509021; LPN C1509021 -> (none); MPN MS9280 -> (none); Manufacturing Part Number (none) -> MS9280
- U1002: LCSC Part Number (none) -> C170157; LPN C170157 -> (none); MPN THS4521IDGKR -> (none); Manufacturing Part Number (none) -> THS4521IDGKR
- U1003: LCSC Part Number (none) -> C2673179; LPN C2673179 -> (none); MPN DGQ2788AEN-T1-GE4 -> (none); Manufacturing Part Number (none) -> DGQ2788AEN-T1-GE4
- U1004: LCSC Part Number (none) -> C7972; LPN C7972 -> (none); MPN LMV321IDBVR -> (none); Manufacturing Part Number (none) -> LMV321IDBVR
- U1005: LCSC Part Number (none) -> C5184435; LPN C5184435 -> (none); MPN TL432 -> (none); Manufacturing Part Number (none) -> TL432

Commit message: order carrier board
Parts:
- L1001: LCSC Part Number C113030 -> C285595; Manufacturing Part Number BLM18SG121TN1D -> UPB160805T-121Y-N
Changed lines of the file:
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@@
 			)
 		)
-		(property "LCSC Part Number" "C113030"
+		(property "LCSC Part Number" "C285595"
 			(at 354.33 53.34 90)
 			(effects
@@
 			)
 		)
-		(property "Manufacturing Part Number" "BLM18SG121TN1D"
+		(property "Manufacturing Part Number" "UPB160805T-121Y-N "
 			(at 354.33 53.34 90)
 			(effects
