File: acoustic-carrier-board/ethernet-phy.kicad_sch (KiCad schematic)
At the start: 49 parts, among them J1201 HR911130A, U1201 KSZ9031RN, Y1201 25MHz

Commit message: added step-files
Parts:
- C1202, C1205, C1208, C1215, C1224: LCSC Part Number (none) -> C19702; LPN C19702 -> (none); MPN CL10A106KP8NNNC -> (none); Manufacturing Part Number (none) -> CL10A106KP8NNNC
- C1203, C1204, C1206, C1207, C1209, C1210, C1216, C1217, C1218, C1219, C1220, C1221, C1222, C1223, C1229: LCSC Part Number (none) -> C22435929; LPN C22435929 -> (none); MPN CGA0201X7R104K160ET -> (none); Manufacturing Part Number (none) -> CGA0201X7R104K160ET
- C1211, C1212, C1213, C1214, C1225: LCSC Part Number (none) -> C285010; LPN C285010 -> (none); MPN 0201B103K250NT -> (none); Manufacturing Part Number (none) -> 0201B103K250NT
- C1226: LCSC Part Number (none) -> C1591; LPN C1591 -> (none); MPN CL10B104KB8NNNC -> (none); Manufacturing Part Number (none) -> CL10B104KB8NNNC
- C1227, C1228: LCSC Part Number (none) -> C1555; LPN C1555 -> (none); MPN 0402CG220J500NT -> (none); Manufacturing Part Number (none) -> 0402CG220J500NT
- D1201: LCSC Part Number (none) -> C2128; LPN C2128 -> (none); MPN 1N4148WS -> (none); Manufacturing Part Number (none) -> 1N4148WS
- J1201: LCSC Part Number (none) -> C54408; LPN C54408 -> (none); MPN HR911130A -> (none); Manufacturing Part Number (none) -> HR911130A
- L1201, L1202, L1203: LCSC Part Number (none) -> C113030; LPN C113030 -> (none); MPN BLM18SG121TN1D -> (none); Manufacturing Part Number (none) -> BLM18SG121TN1D
- R1201: LCSC Part Number (none) -> C17168; LPN C17168 -> (none); MPN 0402WGF0000TCE -> (none); Manufacturing Part Number (none) -> 0402WGF0000TCE
- R1202: LCSC Part Number (none) -> C22790; LPN C22790 -> (none); MPN 0603WAF1202T5E -> (none); Manufacturing Part Number (none) -> 0603WAF1202T5E
- R1203, R1207, R1210, R1211: LCSC Part Number (none) -> C25804; LPN C25804 -> (none); MPN 0603WAF1002T5E -> (none); Manufacturing Part Number (none) -> 0603WAF1002T5E
- R1204, R1208, R1212, R1213: LCSC Part Number (none) -> C25900; LPN C25900 -> (none); MPN 0402WGF4701TCE -> (none); Manufacturing Part Number (none) -> 0402WGF4701TCE
- R1205: LCSC Part Number (none) -> C11702; LPN C11702 -> (none); MPN 0402WGF1001TCE -> (none); Manufacturing Part Number (none) -> 0402WGF1001TCE
- R1206, R1209: LCSC Part Number (none) -> C23179; LPN C23179 -> (none); MPN 0603WAF4700T5E -> (none); Manufacturing Part Number (none) -> 0603WAF4700T5E
- RN1201: LCSC Part Number (none) -> C1980; LPN C1980 -> (none); MPN 4D03WGJ0472T5E -> (none); Manufacturing Part Number (none) -> 4D03WGJ0472T5E
- U1201: LCSC Part Number (none) -> C461575; LPN C461575 -> (none); MPN KSZ9031RNXCC -> (none); Manufacturing Part Number (none) -> KSZ9031RNXCC
- Y1201: LCSC Part Number (none) -> C9006; LPN C9006 -> (none); MPN X322525MOB4SI -> (none); Manufacturing Part Number (none) -> X322525MOB4SI

Commit message: order carrier board
Parts:
- L1201, L1202, L1203: LCSC Part Number C113030 -> C285595; Manufacturing Part Number BLM18SG121TN1D -> UPB160805T-121Y-N
Changed lines of the file:
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@@
 			)
 		)
-		(property "LCSC Part Number" "C113030"
+		(property "LCSC Part Number" "C285595"
 			(at 48.26 45.72 90)
 			(effects
@@
 			)
 		)
-		(property "Manufacturing Part Number" "BLM18SG121TN1D"
+		(property "Manufacturing Part Number" "UPB160805T-121Y-N "
 			(at 48.26 45.72 90)
 			(effects
@@
 			)
 		)
-		(property "LCSC Part Number" "C113030"
+		(property "LCSC Part Number" "C285595"
 			(at 166.37 45.72 90)
 			(effects
@@
 			)
 		)
-		(property "Manufacturing Part Number" "BLM18SG121TN1D"
+		(property "Manufacturing Part Number" "UPB160805T-121Y-N "
 			(at 166.37 45.72 90)
 			(effects
@@
 			)
 		)
-		(property "LCSC Part Number" "C113030"
+		(property "LCSC Part Number" "C285595"
 			(at 105.41 44.45 90)
 			(effects
@@
 			)
 		)
-		(property "Manufacturing Part Number" "BLM18SG121TN1D"
+		(property "Manufacturing Part Number" "UPB160805T-121Y-N "
 			(at 105.41 44.45 90)
 			(effects
