File: acoustic-carrier-board/fpga-bank-01.kicad_sch (KiCad schematic)
At the start: 12 parts, among them IC1 ECP5-BGA256, Y401 Crystal Oscillator

Commit message: added step-files
Parts:
- C401, C402, C404, C405, C407: LCSC Part Number (none) -> C22435929; LPN C22435929 -> (none); MPN CGA0201X7R104K160ET -> (none); Manufacturing Part Number (none) -> CGA0201X7R104K160ET
- C403, C406: LCSC Part Number (none) -> C23733; LPN C23733 -> (none); MPN CL05A475MP5NRNC -> (none); Manufacturing Part Number (none) -> CL05A475MP5NRNC
- IC1: LCSC Part Number (none) -> C1521614; LPN C1521614 -> (none); MPN LFE5U-25F-6BG256C -> (none); Manufacturing Part Number (none) -> LFE5U-25F-6BG256C
- L401: LCSC Part Number (none) -> C113030; LPN C113030 -> (none); MPN BLM18SG121TN1D -> (none); Manufacturing Part Number (none) -> BLM18SG121TN1D
- R401: LCSC Part Number (none) -> C21190; LPN C21190 -> (none); MPN 0603WAF1001T5E -> (none); Manufacturing Part Number (none) -> 0603WAF1001T5E
- Y401: LCSC Part Number (none) -> C496694; LPN C496694 -> (none); MPN O93225100MEDA4SI-13 -> (none); Manufacturing Part Number (none) -> O93225100MEDA4SI-13
Changed lines of the file:
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@@
-			)
-		)
-		(property "LPN" "C22435929"
-			(at 109.22 49.53 0)
-			(effects
-				(font
-					(size 1.27 1.27)
-				)
-				(hide yes)
-			)
-		)
-		(property "MPN" "CGA0201X7R104K160ET "
-			(at 109.22 49.53 0)
-			(effects
-				(font
-					(size 1.27 1.27)
-				)
-				(hide yes)
 			)
 		)
@@
 			)
 		)
-		(property "Check_prices" ""
+		(property "LCSC Part Number" "C22435929"
+			(at 109.22 49.53 0)
+			(effects
+				(font
+					(size 1.27 1.27)
+				)
+				(hide yes)
+			)
+		)
+		(property "Manufacturing Part Number" "CGA0201X7R104K160ET "
 			(at 109.22 49.53 0)
 			(effects
@@
 			)
 		)
-		(property "LPN" "C23733"
-			(at 199.39 48.26 0)
-			(effects
-				(font
-					(size 1.27 1.27)
-				)
-				(hide yes)
-			)
-		)
-		(property "MPN" "CL05A475MP5NRNC"
-			(at 199.39 48.26 0)
-			(effects
-				(font
-					(size 1.27 1.27)
-				)
-				(hide yes)
-			)
-		)
 		(property "Availability" ""
 			(at 199.39 48.26 0)
@@
 			)
 		)
-		(property "Check_prices" ""
+		(property "LCSC Part Number" "C23733"
+			(at 199.39 48.26 0)
+			(effects
+				(font
+					(size 1.27 1.27)
+				)
+				(hide yes)
+			)
+		)
+		(property "Manufacturing Part Number" "CL05A475MP5NRNC"
 			(at 199.39 48.26 0)
 			(effects
@@
 			)
 		)
-		(property "LPN" "C496694"
-			(at 105.41 123.19 0)
-			(effects
-				(font
-					(size 1.27 1.27)
-				)
-				(hide yes)
-			)
-		)
-		(property "MPN" "O93225100MEDA4SI-13"
-			(at 105.41 123.19 0)
-			(effects
-				(font
-					(size 1.27 1.27)
-				)
-				(hide yes)
-			)
-		)
 		(property "Availability" ""
 			(at 105.41 123.19 0)
@@
 			)
 		)
-		(property "Check_prices" ""
+		(property "LCSC Part Number" "C496694"
+			(at 105.41 123.19 0)
+			(effects
+				(font
+					(size 1.27 1.27)
+				)
+				(hide yes)
+			)
+		)
+		(property "Manufacturing Part Number" "O93225100MEDA4SI-13"
 			(at 105.41 123.19 0)
 			(effects
@@
 			)
 		)
-		(property "LPN" "C1521614"
-			(at 335.28 -30.48 0)
-			(effects
-				(font
-					(size 1.27 1.27)
-				)
-				(justify left)
-				(hide yes)
-			)
-		)
-		(property "MPN" "LFE5U-25F-6BG256C "
-			(at 263.144 100.076 0)
+		(property "LCSC Part Number" "C1521614"
+			(at 243.84 100.33 0)
+			(effects
+				(font
+					(size 1.27 1.27)
+				)
+				(hide yes)
+			)
+		)
+		(property "Manufacturing Part Number" "LFE5U-25F-6BG256C "
+			(at 243.84 100.33 0)
 			(effects
 				(font
@@
 			)
 		)
-		(property "LPN" "C22435929"
-			(at 184.15 48.26 0)
-			(effects
-				(font
-					(size 1.27 1.27)
-				)
-				(hide yes)
-			)
-		)
-		(property "MPN" "CGA0201X7R104K160ET "
-			(at 184.15 48.26 0)
-			(effects
-				(font
-					(size 1.27 1.27)
-				)
-				(hide yes)
-			)
-		)
 		(property "Availability" ""
 			(at 184.15 48.26 0)
@@
 			)
 		)
-		(property "Check_prices" ""
+		(property "LCSC Part Number" "C22435929"
+			(at 184.15 48.26 0)
+			(effects
+				(font
+					(size 1.27 1.27)
+				)
+				(hide yes)
+			)
+		)
+		(property "Manufacturing Part Number" "CGA0201X7R104K160ET "
 			(at 184.15 48.26 0)
 			(effects
@@
 			)
 		)
-		(property "LPN" "C23733"
-			(at 124.46 49.53 0)
-			(effects
-				(font
-					(size 1.27 1.27)
-				)
-				(hide yes)
-			)
-		)
-		(property "MPN" "CL05A475MP5NRNC"
-			(at 124.46 49.53 0)
-			(effects
-				(font
-					(size 1.27 1.27)
-				)
-				(hide yes)
-			)
-		)
 		(property "Availability" ""
 			(at 124.46 49.53 0)
@@
 			)
 		)
-		(property "Check_prices" ""
+		(property "LCSC Part Number" "C23733"
+			(at 124.46 49.53 0)
+			(effects
+				(font
+					(size 1.27 1.27)
+				)
+				(hide yes)
+			)
+		)
+		(property "Manufacturing Part Number" "CL05A475MP5NRNC"
 			(at 124.46 49.53 0)
 			(effects
@@
 			)
 		)
-		(property "LPN" "C22435929"
-			(at 116.84 49.53 0)
-			(effects
-				(font
-					(size 1.27 1.27)
-				)
-				(hide yes)
-			)
-		)
-		(property "MPN" "CGA0201X7R104K160ET "
-			(at 116.84 49.53 0)
-			(effects
-				(font
-					(size 1.27 1.27)
-				)
-				(hide yes)
-			)
-		)
 		(property "Availability" ""
 			(at 116.84 49.53 0)
@@
 			)
 		)
-		(property "Check_prices" ""
+		(property "LCSC Part Number" "C22435929"
+			(at 116.84 49.53 0)
+			(effects
+				(font
+					(size 1.27 1.27)
+				)
+				(hide yes)
+			)
+		)
+		(property "Manufacturing Part Number" "CGA0201X7R104K160ET "
 			(at 116.84 49.53 0)
 			(effects
@@
 			)
 		)
-		(property "LPN" "C1521614"
-			(at -22.86 -34.29 0)
-			(effects
-				(font
-					(size 1.27 1.27)
-				)
-				(justify left)
-				(hide yes)
-			)
-		)
-		(property "MPN" "LFE5U-25F-6BG256C "
-			(at 49.276 96.266 0)
+		(property "LCSC Part Number" "C1521614"
+			(at 68.58 96.52 0)
+			(effects
+				(font
+					(size 1.27 1.27)
+				)
+				(hide yes)
+			)
+		)
+		(property "Manufacturing Part Number" "LFE5U-25F-6BG256C "
+			(at 68.58 96.52 0)
 			(effects
 				(font
@@
 			)
 		)
-		(property "LPN" "C113030"
-			(at 127 111.76 90)
-			(effects
-				(font
-					(size 1.27 1.27)
-				)
-				(hide yes)
-			)
-		)
-		(property "MPN" "BLM18SG121TN1D"
-			(at 127 111.76 90)
-			(effects
-				(font
-					(size 1.27 1.27)
-				)
-				(hide yes)
-			)
-		)
 		(property "Availability" ""
 			(at 127 111.76 90)
@@
 			)
 		)
-		(property "Check_prices" ""
+		(property "LCSC Part Number" "C113030"
+			(at 127 111.76 90)
+			(effects
+				(font
+					(size 1.27 1.27)
+				)
+				(hide yes)
+			)
+		)
+		(property "Manufacturing Part Number" "BLM18SG121TN1D"
 			(at 127 111.76 90)
 			(effects
@@
 			)
 		)
-		(property "LPN" "C21190"
-			(at 118.11 123.19 0)
-			(effects
-				(font
-					(size 1.27 1.27)
-				)
-				(hide yes)
-			)
-		)
-		(property "MPN" "0603WAF1001T5E "
-			(at 118.11 123.19 0)
-			(effects
-				(font
-					(size 1.27 1.27)
-				)
-				(hide yes)
-			)
-		)
 		(property "Availability" ""
 			(at 118.11 123.19 90)
@@
 			)
 		)
-		(property "Check_prices" ""
+		(property "LCSC Part Number" "C21190"
+			(at 118.11 123.19 90)
+			(effects
+				(font
+					(size 1.27 1.27)
+				)
+				(hide yes)
+			)
+		)
+		(property "Manufacturing Part Number" "0603WAF1001T5E "
 			(at 118.11 123.19 90)
 			(effects
@@
 			)
 		)
-		(property "LPN" "C22435929"
-			(at 191.77 48.26 0)
-			(effects
-				(font
-					(size 1.27 1.27)
-				)
-				(hide yes)
-			)
-		)
-		(property "MPN" "CGA0201X7R104K160ET "
-			(at 191.77 48.26 0)
-			(effects
-				(font
-					(size 1.27 1.27)
-				)
-				(hide yes)
-			)
-		)
 		(property "Availability" ""
 			(at 191.77 48.26 0)
@@
 			)
 		)
-		(property "Check_prices" ""
+		(property "LCSC Part Number" "C22435929"
+			(at 191.77 48.26 0)
+			(effects
+				(font
+					(size 1.27 1.27)
+				)
+				(hide yes)
+			)
+		)
+		(property "Manufacturing Part Number" "CGA0201X7R104K160ET "
 			(at 191.77 48.26 0)
 			(effects
@@
 			)
 		)
-		(property "LPN" "C22435929"
-			(at 115.57 114.3 0)
-			(effects
-				(font
-					(size 1.27 1.27)
-				)
-				(hide yes)
-			)
-		)
-		(property "MPN" "CGA0201X7R104K160ET "
-			(at 115.57 114.3 0)
-			(effects
-				(font
-					(size 1.27 1.27)
-				)
-				(hide yes)
-			)
-		)
 		(property "Availability" ""
 			(at 115.57 114.3 0)
@@
 			)
 		)
-		(property "Check_prices" ""
+		(property "LCSC Part Number" "C22435929"
+			(at 115.57 114.3 0)
+			(effects
+				(font
+					(size 1.27 1.27)
+				)
+				(hide yes)
+			)
+		)
+		(property "Manufacturing Part Number" "CGA0201X7R104K160ET "
 			(at 115.57 114.3 0)
 			(effects
@@
 			(at 92.71 125.73 0)
 			(effects
-				(font
-					(size 1.27 1.27)
-				)
-				(hide yes)
-			)
-		)
-		(property "Check_prices" ""
-			(at 92.71 125.73 0)
-			(effects

Commit message: order carrier board
Parts:
- L401: LCSC Part Number C113030 -> C285595; Manufacturing Part Number BLM18SG121TN1D -> UPB160805T-121Y-N
Changed lines of the file:
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@@
 			)
 		)
-		(property "LCSC Part Number" "C113030"
+		(property "LCSC Part Number" "C285595"
 			(at 127 111.76 90)
 			(effects
@@
 			)
 		)
-		(property "Manufacturing Part Number" "BLM18SG121TN1D"
+		(property "Manufacturing Part Number" "UPB160805T-121Y-N "
 			(at 127 111.76 90)
 			(effects
